File: Schémas/Tachymetre.kicad_pcb (KiCad board)
At the start: 2 copper layers, 79 x 40 mm, 10 parts, among them J1 Conn_01x05, J3 Conn_01x04

Commit message: Repère Oled
Other:
- board text added: "5V"
- board text added: "GND"
- board text added: "SCL"
- board text added: "SDA"
