File: Schémas/Tachymetre.sch (KiCad schematic (older format))
At the start: 10 parts, among them J1 Conn_01x05, J3 Conn_01x04

Commit message: Commentaires
Other:
- note added: "Alimentation"
- note added: "Capteur"
- moved on the sheet: C1, C2, D1, J1, J3, L1, R100, R101, VR1
